File: Voyager60.sch (KiCad schematic (older format))
At the start: 201 parts, among them SW1 5.2x5.2mm, U1 ATmega32U4-MU, U2 PRTR5V0U2X, Y1 16Mhz

Commit message: Clean up rescued symbols in the schematic; get rid or all ERC errors/warnings
Parts:
- removed K_ESC2: MX-1U, MX_Alps_Hybrid:ALPS-1U, symbol MX_Alps_Hybrids:MX-1U
- added K_#5: MX-1U, MX_Alps_Hybrid:ALPS-1U, symbol Switch:SW_Push_45deg
- K_#1: renamed from K_#2; symbol MX_Alps_Hybrids:MX-1U -> Switch:SW_Push_45deg
- K_#10, K_#6, K_#7, K_#8, K_#9, K_'1, K_,1, K_-1, K_.1, K_/1, K_;1, K_=1, K_A1, K_ALT1, K_ALT2, K_ALT3, K_B1, K_BACK1, K_C1, K_CAPS1, K_CAPS2, K_CAPS3, K_CTRL1, K_CTRL2, K_D1, K_E1, K_ENTER1, K_ENTER2, K_ENTER3, K_ENTER4, K_F1, K_G1, K_H1, K_I1, K_J1, K_K1, K_L1, K_M1, K_N1, K_O1, K_P1, K_Q1, K_R1, K_RALT1, K_RALT2, K_RALT3, K_RCTRL2, K_RCTRL3, K_RMENU2, K_RSHIFT1, K_RWIN1, K_RWIN2, K_RWIN3, K_S1, K_SBACK1, K_SBACK2, K_SHIFT1, K_SHIFT2, K_SHIFT3, K_SPACE1, K_SPACE2, K_SPACE3, K_SPACE4, K_SPACE5, K_SRSHIFT1, K_SRSHIFT2, K_T1, K_TAB1, K_U1, K_V1, K_W1, K_WIN1, K_WIN2, K_WIN3, K_X1, K_Y1, K_Z1, K_[1, K_\1, K_\2, K_]1: symbol MX_Alps_Hybrids:MX-1U -> Switch:SW_Push_45deg
- K_#2: renamed from K_#3; symbol MX_Alps_Hybrids:MX-1U -> Switch:SW_Push_45deg
- K_#3: renamed from K_#4; symbol MX_Alps_Hybrids:MX-1U -> Switch:SW_Push_45deg
- K_#4: renamed from K_#5; symbol MX_Alps_Hybrids:MX-1U -> Switch:SW_Push_45deg
- K_ESC1: renamed from K_#1; symbol MX_Alps_Hybrids:MX-1U -> Switch:SW_Push_45deg
- K_ESC2: renamed from K_ESC1; symbol MX_Alps_Hybrids:MX-1U -> Switch:SW_Push_45deg
- SW1: symbol Voyager60-rescue:SW_Push -> Switch:SW_Push
- U1: symbol Voyager60-rescue:ATmega32U4-MU-MCU_Microchip_ATmega -> MCU_Microchip_ATmega:ATmega32U4-MU
Connections:
- wire segments 646 -> 511
- no-connect marks 2 -> 9
