File: Voyager60.kicad_pcb (KiCad board)
At the start: 2 copper layers, 285 x 95.1 mm, 205 parts, among them SW1 5.2x5.2mm, U1 ATmega32U4-MU, U2 PRTR5V0U2X, Y1 16Mhz

Commit message: Redo layout with SMK footprints
Parts:
- removed D58, D62: SOD-123, Diodes_SMD:D_SOD-123
- removed the K_#3 at (88.9, 31.8)
- removed K_ENTER4, K_ESC2: MX-1U, MX_Alps_Hybrid:ALPS-1U
- removed K_SPACE3: MX-2.25U, MX_Alps_Hybrid:ALPS-2.25U
- removed K_SPACE4: MX-2.75U, MX_Alps_Hybrid:ALPS-2.75U
- removed K_SPACE5: MX-1.25U, MX_Alps_Hybrid:ALPS-1.25U
- added K_#4: MX-1U, smk:SW_SMK, F.Cu at (108.0, 31.8)
- K_#1, K_#10, K_#2, K_#5, K_#6, K_#7, K_#8, K_#9, K_'1, K_,1, K_-1, K_.1, K_/1, K_;1, K_=1, K_A1, K_B1, K_C1, K_D1, K_E1, K_ENTER3, K_ESC1, K_F1, K_G1, K_H1, K_I1, K_J1, K_K1, K_L1, K_M1, K_N1, K_O1, K_P1, K_Q1, K_R1, K_RWIN3, K_S1, K_SBACK1, K_SBACK2, K_SHIFT3, K_SRSHIFT2, K_T1, K_U1, K_V1, K_W1, K_WIN2, K_X1, K_Y1, K_Z1, K_[1, K_\2, K_]1: footprint MX_Alps_Hybrid:ALPS-1U -> smk:SW_SMK
- K_#3: renamed from K_#4; footprint MX_Alps_Hybrid:ALPS-1U -> smk:SW_SMK
- K_ALT1, K_CAPS2, K_CTRL1, K_RALT2, K_RCTRL2, K_RMENU2, K_RWIN1, K_RWIN2, K_SHIFT2, K_WIN1, K_WIN3: footprint MX_Alps_Hybrid:ALPS-1.25U -> smk:SW_SMK
- K_ALT2, K_ALT3, K_CAPS3, K_CTRL2, K_RALT1, K_RALT3, K_RCTRL3, K_TAB1, K_\1: footprint MX_Alps_Hybrid:ALPS-1.5U -> smk:SW_SMK
- K_BACK1: footprint MX_Alps_Hybrid:ALPS-2U -> smk:SW_SMK_2u
- K_CAPS1, K_SRSHIFT1: footprint MX_Alps_Hybrid:ALPS-1.75U -> smk:SW_SMK
- K_ENTER1, K_SHIFT1: footprint MX_Alps_Hybrid:ALPS-2.25U -> smk:SW_SMK_2u
- K_ENTER2: value MX-1U -> MX-2U; footprint MX_Alps_Hybrid:ALPS-1U -> smk:SW_SMK_2u_R
- K_RSHIFT1: footprint MX_Alps_Hybrid:ALPS-2.75U -> smk:SW_SMK_2u
- K_SPACE1: footprint MX_Alps_Hybrid:ALPS-7U -> smk:SW_SMK_7u_R
- K_SPACE2: footprint MX_Alps_Hybrid:ALPS-6.25U -> smk:SW_SMK_6.25u_R
- SW1: footprint Molex-0548190589:SKQG-1155865 -> Button_Switch_SMD:SW_SPST_SKQG_WithStem
- U1: footprint Housings_DFN_QFN:QFN-44-1EP_7x7mm_Pitch0.5mm -> Package_DFN_QFN:QFN-44-1EP_7x7mm_P0.5mm_EP5.2x5.2mm
- moved D61 34.1 mm to (173.8, 105.0)
- moved K_#3 19.0 mm to (88.9, 31.8)
- moved D1 12.7 mm to (28.6, 41.7), turned to 180 degrees
- moved D29 7.50 mm to (300.9, 55.9), turned to 0 degrees
- moved C15 6.76 mm to (289.1, 92.9), turned to 0 degrees
- moved C7 6.45 mm to (46.9, 66.0), turned to 180 degrees
- moved C17 5.28 mm to (217.1, 97.5)
- moved RGB6 5.28 mm to (211.6, 97.5)
- moved K_ENTER3 4.76 mm to (293.7, 60.3), turned to 90 degrees
- moved D44 3.22 mm to (66.7, 86.0)
- moved D45 3.22 mm to (63.5, 86.0)
- moved C8 2.54 mm to (46.9, 71.9)
- moved R74 2.50 mm to (48.6, 34.0)
- moved Y1 2.22 mm to (46.9, 69.0)
- moved R70 1.52 mm to (48.8, 75.8)
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Connections:
- K_#3 pad 1: COL4 -> COL3
- K_#3 pad 2: Net-(D5-Pad2) -> Net-(D4-Pad2)
- K_ENTER1 pad 1: COL13 -> Net-(D43-Pad2)
- K_ENTER1 pad 2: Net-(D43-Pad2) -> COL13
- K_SHIFT2 pad 1: COL0 -> Net-(D45-Pad2)
- K_SHIFT2 pad 2: Net-(D45-Pad2) -> COL0
- K_SRSHIFT2 pad 1: COL13 -> Net-(D57-Pad2)
- K_SRSHIFT2 pad 2: Net-(D57-Pad2) -> COL13
- K_\2 pad 1: COL13 -> Net-(D29-Pad2)
- K_\2 pad 2: Net-(D29-Pad2) -> COL13
- RGB14 pad 2: Net-(RGB14-Pad2) -> (no net)
- U1 pad 1: Net-(U1-Pad1) -> (no net)
- U1 pad 12: Net-(U1-Pad12) -> (no net)
- U1 pad 18: Net-(U1-Pad18) -> (no net)
- U1 pad 19: Net-(U1-Pad19) -> (no net)
- U1 pad 42: Net-(U1-Pad42) -> (no net)
- U1 pad 8: Net-(U1-Pad8) -> (no net)
- USB1 pad 3: Net-(USB1-Pad3) -> (no net)
- USB1 pad 9: Net-(USB1-Pad9) -> (no net)
Routing:
- net +5V: track 757.3 -> 702.0 mm, vias 8 -> 7
- net COL4: track 266.8 -> 232.0 mm
- net COL8: track 375.1 -> 351.4 mm
- net COL13: track 376.7 -> 399.6 mm
- net COL0: track 145.8 -> 129.4 mm
- net ROW3: track 303.2 -> 287.0 mm
- net Net-(D1-Pad2): track 21.1 -> 6.01 mm
- net COL3: track 188.2 -> 173.3 mm
- net COL5: track 303.7 -> 288.9 mm
- net Net-(D44-Pad2): track 5.63 -> 18.8 mm, vias 0 -> 1
- net COL6: track 395.5 -> 382.6 mm
- net Net-(D61-Pad2): track 31.4 -> 18.5 mm
- net Net-(D29-Pad2): track 37.5 -> 50.1 mm, vias 1 -> 0
- net ROW4: track 318.6 -> 306.6 mm
- net ROW0: track 325.7 -> 313.9 mm
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